Commit message: add openagv_bringup package

File: catkin_ws/src/openagv_description/urdf/openagv.urdf (robot description, URDF)
Before this commit: robot OpenAGV, 5 links, 4 joints
Links:
- removed link kinect_link
- added link camera_link; visual box size=0.06150 0.275386 0.038
Joints:
- removed joint kinect_joint
- added joint camera_joint: type fixed, parent base_link, child camera_link, origin xyz=0.051306 0 0.19087 rpy=0 0 0
